Commit message: 🌱init commit: 初期コミット

File: orne_box_description/urdf/orne_box.gazebo.xacro (robot description, xacro)
@@ -1,18 +1,27 @@
 <?xml version="1.0"?>
-<robot name="orne_box" xmlns:xacro="http://ros.org/wiki/xacro">
+<robot xmlns:xacro="http://ros.org/wiki/xacro" name="orne_box">
   <xacro:property name="PI" value="3.1415926535897931"/>
   <xacro:arg name="laser_visual" default="true"/>
-  <xacro:arg name="imu_visual"   default="false"/>
-  <gazebo>
-    <plugin name="gazebo_ros_control" filename="libgazebo_ros_control.so">
-      <robotSimType>icart_mini_gazebo/ICartMiniHWSim</robotSimType>
-    </plugin>
+  <xacro:arg name="imu_visual" default="false"/>
+  <xacro:arg name="enable_camera" default="false"/>
+  <gazebo reference="left_caster_wheel_link">
+    <mu1>0.75</mu1>
+    <mu2>0.75</mu2>
+    <kp>1000000.0</kp>
+    <kd>100.0</kd>
+    <minDepth>0.001</minDepth>
+    <maxVel>1.0</maxVel>
   </gazebo>
-  <gazebo reference="base_link">
-    <material>Gazebo/Orange</material>
+  <gazebo reference="right_caster_wheel_link">
+    <mu1>0.75</mu1>
+    <mu2>0.75</mu2>
+    <kp>1000000.0</kp>
+    <kd>100.0</kd>
+    <minDepth>0.001</minDepth>
+    <maxVel>1.0</maxVel>
   </gazebo>
-  <gazebo reference="wheel_left_link">
-    <mu1>1.0</mu1>
-    <mu2>1.0</mu2>
+  <gazebo reference="left_wheel">
+    <mu1>0.85</mu1>
+    <mu2>0.85</mu2>
     <kp>1000000.0</kp>
     <kd>100.0</kd>
@@ -21,7 +30,7 @@
     <material>Gazebo/White</material>
   </gazebo>
-  <gazebo reference="wheel_right_link">
-    <mu1>1.0</mu1>
-    <mu2>1.0</mu2>
+  <gazebo reference="right_wheel">
+    <mu1>0.85</mu1>
+    <mu2>0.85</mu2>
     <kp>1000000.0</kp>
     <kd>100.0</kd>
@@ -30,51 +39,152 @@
     <material>Gazebo/White</material>
   </gazebo>
-  <gazebo reference="caster_front_link">
-    <mu1>0.0</mu1>
-    <mu2>0.0</mu2>
-    <material>Gazebo/Red</material>
-  </gazebo>
-  <gazebo reference="imu_link">
-    <sensor type="imu" name="imu">
-      <always_on>true</always_on>
-      <visualize>$(arg imu_visual)</visualize>
-    </sensor>
-    <material>Gazebo/FlatBlack</material>
-  </gazebo>
-  <!-- hokuyo -->
-  <gazebo reference="hokuyo_link">
-    <sensor type="ray" name="head_hokuyo_sensor">
-      <pose>0 0 0 0 0 0</pose>
-      <visualize>$(arg laser_visual)</visualize>
-      <update_rate>40</update_rate>
-      <ray>
-        <scan>
-          <horizontal>
-            <samples>880</samples>
-            <resolution>0.25</resolution>
-            <min_angle>${-PI/180*110}</min_angle>
-            <max_angle>${ PI/180*110}</max_angle>
-          </horizontal>
-        </scan>
-        <range>
-          <min>0.10</min>
-          <max>30.0</max>
-          <resolution>0.01</resolution>
-        </range>
-        <noise>
-          <type>gaussian</type>
-          <!-- Noise parameters based on published spec for Hokuyo laser
-               achieving "+-30mm" accuracy at range < 10m.  A mean of 0.0m and
-               stddev of 0.01m will put 99.7% of samples within 0.03m of the true
-               reading. -->
-          <mean>0.0</mean>
-          <stddev>0.01</stddev>
-        </noise>
-      </ray>
-      <plugin name="gazebo_ros_head_hokuyo_controller" filename="libgazebo_ros_laser.so">
-        <topicName>/scan</topicName>
-        <frameName>hokuyo_link</frameName>
+  <!-- @TODO More clear boolean operation -->
+    <!-- <gazebo>
+      <plugin name="gazebo_ros_control" filename="libgazebo_ros_control.so">
+        <robotNamespace>orne_box</robotNamespace>
+        <robotSimType>gazebo_ros_control/DefaultRobotHWSim</robotSimType>
       </plugin>
-    </sensor>
-  </gazebo>
+    </gazebo> -->
+    <gazebo>
+      <plugin name="gazebo_ros_control" filename="libgazebo_ros_diff_drive.so">
+        <always_on>true</always_on>
+        <robotNamespace>/orne_box</robotNamespace>
+        <!-- frame and cmd_vel -->
+        <command_topic>cmd_vel</command_topic>
+        <odometry_topic>odom</odometry_topic>
+        <odometry_frame>odom</odometry_frame>
+        <!-- <odometrySource>world</odometrySource> -->
+        <robot_base_frame>base_footprint</robot_base_frame>
+        <update_rate>30</update_rate>
+        <!-- wheels -->
+        <left_joint>left_wheel_joint</left_joint>
+        <right_joint>right_wheel_joint</right_joint>
+        <!-- kinematics -->
+        <wheel_separation>0.46</wheel_separation>
+        <wheel_diameter>0.304</wheel_diameter>
+        <wheel_acceleration>1</wheel_acceleration>
+        <max_wheel_torque>20</max_wheel_torque>
+        <max_wheel_acceleration>1.0</max_wheel_acceleration>
+        <!-- output -->
+        <publish_odom>true</publish_odom>
+        <publish_odom_tf>true</publish_odom_tf>
+        <publish_wheel_tf>false</publish_wheel_tf>
+      </plugin>
+    </gazebo>
+    <gazebo reference="base_link">
+      <material>Gazebo/Orange</material>
+    </gazebo>
+    <!-- imu -->
+    <gazebo reference="imu_link">
+      <sensor type="imu" name="imu">
+        <plugin filename="libgazebo_ros_imu_sensor.so" name="imu_plugin">
+          <ros>
+            <remapping>~/out:=imu</remapping>
+          </ros>
+          <initial_orientation_as_reference>false</initial_orientation_as_reference>
+        </plugin>
+        <always_on>true</always_on>
+        <update_rate>100</update_rate>
+        <visualize>true</visualize>
+        <imu>
+        <angular_velocity>
+          <x>
+            <noise type="gaussian">
+                <mean>0.0</mean>
+                <stddev>2e-4</stddev>
+                <bias_mean>0.0000075</bias_mean>
+                <bias_stddev>0.0000008</bias_stddev>
+              </noise>
+            </x>
+            <y>
+              <noise type="gaussian">
+                <mean>0.0</mean>
+                <stddev>2e-4</stddev>
+                <bias_mean>0.0000075</bias_mean>
+                <bias_stddev>0.0000008</bias_stddev>
+              </noise>
+            </y>
+            <z>
+              <noise type="gaussian">
+                <mean>0.0</mean>
+                <stddev>2e-4</stddev>
+                <bias_mean>0.0000075</bias_mean>
+                <bias_stddev>0.0000008</bias_stddev>
+              </noise>
+            </z>
+          </angular_velocity>
+          <linear_acceleration>
+            <x>
+              <noise type="gaussian">
+                <mean>0.0</mean>
+                <stddev>1.7e-2</stddev>
+                <bias_mean>0.1</bias_mean>
+                <bias_stddev>0.001</bias_stddev>
+              </noise>
+            </x>
+            <y>
+              <noise type="gaussian">
+                <mean>0.0</mean>
+                <stddev>1.7e-2</stddev>
+                <bias_mean>0.1</bias_mean>
+                <bias_stddev>0.001</bias_stddev>
+              </noise>
+            </y>
+            <z>
+              <noise type="gaussian">
+                <mean>0.0</mean>
+                <stddev>1.7e-2</stddev>
+                <bias_mean>0.1</bias_mean>
+                <bias_stddev>0.001</bias_stddev>
+              </noise>
+            </z>
+          </linear_acceleration>
+        </imu>
+      </sensor>
+      <material>Gazebo/Green</material>
+    </gazebo>
+    <!-- hokuyo -->
+    <gazebo reference="hokuyo_link">
+      <sensor type="ray" name="head_hokuyo_sensor">
+        <pose>0 0 0 0 0 0</pose>
+        <visualize>$(arg laser_visual)</visualize>
+        <update_rate>40</update_rate>
+        <ray>
+          <scan>
+            <horizontal>
+              <samples>880</samples>
+              <resolution>0.25</resolution>
+              <min_angle>${-PI/180*110}</min_angle>
+              <max_angle>${ PI/180*110}</max_angle>
+            </horizontal>
+            <vertical>
+              <samples>1</samples>
+              <resolution>1</resolution>
+            </vertical>
+          </scan>
+          <range>
+            <min>0.10</min>
+            <max>30.0</max>
+            <resolution>0.01</resolution>
+          </range>
+          <noise>
+            <type>gaussian</type>
+            <!-- Noise parameters based on published spec for Hokuyo laser
+                 achieving "+-30mm" accuracy at range < 10m.  A mean of 0.0m and
+                 stddev of 0.01m will put 99.7% of samples within 0.03m of the true
+                 reading. -->
+            <mean>0.0</mean>
+            <stddev>0.01</stddev>
+          </noise>
+        </ray>
+        <plugin name="gazebo_ros_head_hokuyo_controller" filename="libgazebo_ros_ray_sensor.so">
+          <ros>
+            <remapping>~/out:=scan</remapping>
+          </ros>
+          <frame_name>hokuyo_link</frame_name>
+          <output_type>sensor_msgs/LaserScan</output_type>
+        </plugin>
+      </sensor>
+      <material>Gazebo/Black</material>
+    </gazebo>
 </robot>

File: orne_box_description/urdf/orne_box.urdf.xacro (robot description, xacro)
@@ -1,207 +1,61 @@
-<?xml version="1.0" ?>
-<robot name="orne_box" xmlns:xacro="http://www.ros.org/wiki/xacro">
+<?xml version="1.0"?>
+<robot xmlns:xacro="http://www.ros.org/wiki/xacro" name="orne_box">
   <xacro:property name="PI" value="3.1415926535897931"/>
-  <xacro:include filename="$(find icart_mini_description)/urdf/materials.xacro" />
+  <xacro:include filename="$(find orne_box_description)/urdf/material_colors.xacro"/>
   <xacro:include filename="$(find orne_box_description)/urdf/orne_box.gazebo.xacro"/>
-  <link name="base_link">
-<!--
-    <visual>
-      <origin xyz="0 0 -0.154" rpy="0 0 0"/>
-      <geometry>
-        <mesh filename="package://orne_box_description/meshes/bases/orne_box_base.stl" scale="1 1 1"/>
-      </geometry>
-      <material name="orange"/>
-    </visual>
--->
-    <visual>
-      <origin xyz="0.090 0 0.1715" rpy="0 0 0"/>
-      <geometry>
-        <box size="0.400 0.404 0.202"/>
-      </geometry>
-      <material name="orange"/>
-    </visual>
-    <visual>
-      <origin xyz="0.36125 0 0.2625" rpy="0 0 0"/>
-      <geometry>
-        <box size="0.1425 0.404 0.020"/>
-      </geometry>
-      <material name="orange"/>
-    </visual>
-    <visual>
-      <origin xyz="0.35625 0 0.156" rpy="0 0 0"/>
-      <geometry>
-        <box size="0.1325 0.404 0.020"/>
-      </geometry>
-      <material name="orange"/>
-    </visual>
-    <visual>
-      <origin xyz="-0.120 0 0.4815" rpy="0 0 0"/>
-      <geometry>
-        <box size="0.020 0.404 0.822"/>
-      </geometry>
-      <material name="orange"/>
-    </visual>
-    <collision>
-      <origin xyz="0.090 0 0.1715" rpy="0 0 0"/>
-      <geometry>
-        <box size="0.400 0.404 0.202"/>
-      </geometry>
-    </collision>
-    <collision>
-      <origin xyz="0.36125 0 0.2625" rpy="0 0 0"/>
-      <geometry>
-        <box size="0.1425 0.404 0.020"/>
-      </geometry>
-    </collision>
-    <collision>
-      <origin xyz="0.35625 0 0.156" rpy="0 0 0"/>
-      <geometry>
-        <box size="0.1325 0.404 0.020"/>
-      </geometry>
-    </collision>
-    <collision>
-      <origin xyz="-0.120 0 0.4815" rpy="0 0 0"/>
-      <geometry>
-        <box size="0.020 0.404 0.822"/>
-      </geometry>
-    </collision>
-    <inertial>
-      <origin xyz="0.090 0 0.1715" rpy="0 0 0"/>
-      <mass value="25.0"/>
-      <inertia ixx="1.0" ixy="0.0" ixz="0.0" iyy="1.0" iyz="0.0" izz="1.0" />
-    </inertial>
-  </link>
-  <joint name="left_wheel_hinge" type="revolute">
-    <parent link="base_link"/>
-    <child link="wheel_left_link"/>
+  <xacro:include filename="$(find orne_box_description)/urdf/links/base_link.urdf.xacro"/>
+  <xacro:include filename="$(find orne_box_description)/urdf/links/caster_wheel_link.urdf.xacro"/>
+  <xacro:include filename="$(find orne_box_description)/urdf/links/caster_swivel_link.urdf.xacro"/>
+  <xacro:include filename="$(find orne_box_description)/urdf/links/wheel_link.urdf.xacro"/>
+  <xacro:include filename="$(find orne_box_description)/urdf/joints/caster_wheel_joint.urdf.xacro"/>
+  <xacro:include filename="$(find orne_box_description)/urdf/joints/caster_swivel_joint.urdf.xacro"/>
+  <xacro:include filename="$(find orne_box_description)/urdf/joints/wheel_joint.urdf.xacro"/>
+  <xacro:include filename="$(find orne_box_description)/urdf/sensors/imu.urdf.xacro"/>
+  <xacro:include filename="$(find orne_box_description)/urdf/sensors/hokuyo.urdf.xacro"/>
+  <!-- Setting for base -->
+  <xacro:base_link/>
+  <!-- Setting for caster -->
+  <xacro:caster_wheel_link prefix="left"/>
+  <xacro:caster_swivel_link prefix="left"/>
+  <xacro:caster_wheel_joint prefix="left"/>
+  <xacro:caster_swivel_joint prefix="left" parent="base_link">
+    <origin xyz="0.362 0.150 0.115" rpy="0 0 0"/>
+  </xacro:caster_swivel_joint>
+  <xacro:caster_wheel_link prefix="right"/>
+  <xacro:caster_swivel_link prefix="right"/>
+  <xacro:caster_wheel_joint prefix="right"/>
+  <xacro:caster_swivel_joint prefix="right" parent="base_link">
+    <origin xyz="0.362 -0.150 0.115" rpy="0 0 0"/>
+  </xacro:caster_swivel_joint>
+  <!-- Setting for left wheel -->
+  <xacro:wheel_joint prefix="left" parent="base_link">
     <origin xyz="0.0 0.23075 0.152" rpy="${-PI/2} 0 0"/>
     <axis xyz="0 0 1"/>
-    <limit effort="100" velocity="100.0"  lower="-5000" upper="5000" />
-  </joint>
-  <link name="wheel_left_link">
-    <visual>
-      <origin xyz="0 0 0" rpy="0 0 0"/>
-      <geometry>
-        <mesh filename="package://orne_box_description/meshes/wheels/tire.stl" scale="1 1 1"/>
-      </geometry>
-<!--
-      <origin xyz="0 0 0" rpy="0 0 0"/>
-      <geometry>
-        <cylinder length="0.045" radius="0.152"/>
-      </geometry>
--->
-      <material name="white"/>
-    </visual>
-    <collision>
-      <origin xyz="0 0 0" rpy="0 0 0"/>
-      <geometry>
-        <cylinder length="0.045" radius="0.152"/>
-      </geometry>
-    </collision>
-    <inertial>
-      <origin xyz="0 0 0" />
-      <mass value="0.2" />
-      <inertia ixx="0.1" ixy="0.0" ixz="0.0" iyy="0.1" iyz="0.0" izz="0.1" />
-    </inertial>
-  </link>
-  <joint name="right_wheel_hinge" type="revolute">
-    <parent link="base_link"/>
-    <child link="wheel_right_link"/>
+  </xacro:wheel_joint>
+  <xacro:wheel_link prefix="left" width="0.045" radius="0.152">
+    <origin xyz="0.0 0.0 0.0" rpy="0 0 0"/>
+  </xacro:wheel_link>
+  <!-- Setting for right wheel -->
+  <xacro:wheel_joint prefix="right" parent="base_link">
     <origin xyz="0.0 -0.23075 0.152" rpy="${-PI/2} 0 0"/>
     <axis xyz="0 0 1"/>
-    <limit effort="100" velocity="100.0"  lower="-5000" upper="5000" />
-  </joint>
-  <link name="wheel_right_link">
-    <visual>
-      <origin xyz="0 0 0" rpy="0 0 0"/>
-      <geometry>
-        <mesh filename="package://orne_box_description/meshes/wheels/tire.stl" scale="1 1 1"/>
-      </geometry>
-<!--
-      <origin xyz="0 0 0" rpy="0 0 0"/>
-      <geometry>
-        <cylinder length="0.045" radius="0.152"/>
-      </geometry>
--->
-      <material name="white"/>
-    </visual>
-    <collision>
-      <origin xyz="0 0 0" rpy="0 0 0"/>
-      <geometry>
-        <cylinder length="0.045" radius="0.152"/>
-      </geometry>
-    </collision>
-    <inertial>
-      <origin xyz="0 0 0" />
-      <mass value="0.2" />
-      <inertia ixx="0.1" ixy="0.0" ixz="0.0" iyy="0.1" iyz="0.0" izz="0.1" />
-    </inertial>
-  </link>
-  <joint name="caster_front_joint" type="fixed">
-    <parent link="base_link"/>
-    <child link="caster_front_link"/>
-    <origin xyz="0.362 0 0.050" rpy="0 0 0"/>
-  </joint>
-  <link name="caster_front_link">
-    <visual>
-      <origin xyz="0 0.150 0" rpy="${PI/2} 0 0"/>
-      <geometry>
-        <cylinder length="0.025" radius="0.050"/>
-      </geometry>
-      <material name="red"/>
-    </visual>
-    <visual>
-      <origin xyz="0 -0.150 0" rpy="${PI/2} 0 0"/>
-      <geometry>
-        <cylinder length="0.025" radius="0.050"/>
-      </geometry>
-      <material name="red"/>
-    </visual>
-    <collision>
-      <origin xyz="0 0.150 0" rpy="${PI/2} 0 0"/>
-      <geometry>
-        <cylinder length="0.025" radius="0.050"/>
-      </geometry>
-    </collision>
-    <collision>
-      <origin xyz="0 -0.150 0" rpy="${PI/2} 0 0"/>
-      <geometry>
-        <cylinder length="0.025" radius="0.050"/>
-      </geometry>
-    </collision>
-    <inertial>
-      <origin xyz="0 0 0" />
-      <mass value="0.2" />
-      <inertia ixx="0.1" ixy="0.0" ixz="0.0" iyy="0.1" iyz="0.0" izz="0.1" />
-    </inertial>
-  </link>
-  <xacro:include filename="$(find icart_mini_description)/urdf/sensors/imu.urdf.xacro"/>
-  <!-- Setting for imu -->
+  </xacro:wheel_joint>
+  <xacro:wheel_link prefix="right" width="0.045" radius="0.152">
+    <origin xyz="0.0 0.0 0.0" rpy="0 0 0"/>
+  </xacro:wheel_link>
+  <!-- Setting for IMU -->
+  <!-- <xacro:sensor_imu name="imu" parent="base_link" size="0.05 0.05 0.05">
+    <origin xyz="0.23 0.0 0.270" rpy="${-PI} 0 ${PI/2}"/>
+  </xacro:sensor_imu> -->
   <xacro:sensor_imu name="imu" parent="base_link" size="0.05 0.05 0.05">
-    <origin xyz="0.3 0 0.2445" rpy="0 0 ${-PI/2}"/>
+    <origin xyz="0.23 0.0 0.270" rpy="0 0 0"/>
+    <origin_child xyz="0.0 0.0 0.0" rpy="0 0 0"/>
   </xacro:sensor_imu>
-  <xacro:include filename="$(find icart_mini_description)/urdf/sensors/hokuyo.urdf.xacro"/>
-  <xacro:sensor_hokuyo name="hokuyo" parent="base_link">
+  <!-- Setting for 2D-LiDAR -->
+  <xacro:sensor_hokuyo name="hokuyo" parent="base_link" size="0.05 0.05 0.05">
     <origin xyz="0.374295 0 0.2185" rpy="${-PI} 0 0"/>
   </xacro:sensor_hokuyo>
-  <transmission name="tran1">
-    <type>transmission_interface/SimpleTransmission</type>
-    <joint name="left_wheel_hinge">
-      <hardwareInterface>VelocityJointInterface</hardwareInterface>
-    </joint>
-  <actuator name="left_motor">
-      <hardwareInterface>VelocityJointInterface</hardwareInterface>
-      <mechanicalReduction>1</mechanicalReduction>
-    </actuator>
-  </transmission>
-  <transmission name="tran2">
-    <type>transmission_interface/SimpleTransmission</type>
-    <joint name="right_wheel_hinge">
-      <hardwareInterface>VelocityJointInterface</hardwareInterface>
-    </joint>
-  <actuator name="right_motor">
-      <hardwareInterface>VelocityJointInterface</hardwareInterface>
-      <mechanicalReduction>1</mechanicalReduction>
-    </actuator>
-  </transmission>
+  <xacro:sensor_hokuyo name="mirror_lidar" parent="base_link" size="0.05 0.05 0.05">
+    <origin xyz="0.43 0.0 0.34" rpy="0 0.314 0"/>
+  </xacro:sensor_hokuyo>
 </robot>

Commit message: 🐛fix: sim

File: orne_box_description/urdf/orne_box.gazebo.xacro (robot description, xacro)
@@ -80,5 +80,5 @@
         <plugin filename="libgazebo_ros_imu_sensor.so" name="imu_plugin">
           <ros>
-            <remapping>~/out:=imu</remapping>
+            <remapping>~/out:=imu/data</remapping>
           </ros>
           <initial_orientation_as_reference>false</initial_orientation_as_reference>

File: orne_box_description/urdf/orne_box.urdf.xacro (robot description, xacro)
@@ -54,5 +54,5 @@
   <!-- Setting for 2D-LiDAR -->
   <xacro:sensor_hokuyo name="hokuyo" parent="base_link" size="0.05 0.05 0.05">
-    <origin xyz="0.374295 0 0.2185" rpy="${-PI} 0 0"/>
+    <origin xyz="0.374295 0 0.2185" rpy="0 0 0"/>
   </xacro:sensor_hokuyo>
   <xacro:sensor_hokuyo name="mirror_lidar" parent="base_link" size="0.05 0.05 0.05">
