Commit message: 🐛fix: hokuyo

File: orne_box_description/urdf/orne_box.urdf.xacro (robot description, xacro)
@@ -54,8 +54,8 @@
   <!-- Setting for 2D-LiDAR -->
   <xacro:sensor_hokuyo name="hokuyo" parent="base_link" size="0.05 0.05 0.05">
-    <origin xyz="0.374295 0 0.2185" rpy="0 0 0"/>
+    <origin xyz="0.364295 0 0.185" rpy="3.14 0 0"/>
   </xacro:sensor_hokuyo>
-  <xacro:sensor_hokuyo name="mirror_lidar" parent="base_link" size="0.05 0.05 0.05">
+  <!-- <xacro:sensor_hokuyo name="mirror_lidar" parent="base_link" size="0.05 0.05 0.05">
     <origin xyz="0.43 0.0 0.34" rpy="0 0.314 0"/>
-  </xacro:sensor_hokuyo>
+  </xacro:sensor_hokuyo> -->
 </robot>
