Commit message: 🔧modify: rfans位置修正

File: orne_box_description/urdf/orne_box_3d_lidar_rfans.urdf.xacro (robot description, xacro)
@@ -8,5 +8,6 @@
     <!-- Setting for 3D-LiDAR -->
     <xacro:VLP-16 parent="base_link" name="surestar" topic="/rfans_points" organize_cloud="false" hz="10" samples="440" gpu="false">
-      <origin xyz="0.23 0 0.40" rpy="0 0 3.14"/>
+      <!-- <origin xyz="0.23 0 0.40" rpy="0 0 3.14"/> -->
+      <origin xyz="-0.1 0 0.6" rpy="0 0 3.14"/>
     </xacro:VLP-16>
   </xacro:if>

Commit message: 🐛fix: urdf

File: orne_box_description/urdf/orne_box_3d_lidar_rfans.urdf.xacro (robot description, xacro)
@@ -8,5 +8,5 @@
     <!-- Setting for 3D-LiDAR -->
     <xacro:VLP-16 parent="base_link" name="surestar" topic="/rfans_points" organize_cloud="false" hz="10" samples="440" gpu="false">
-      <origin xyz="0.23 0 0.40" rpy="0 0 0"/>
+      <origin xyz="-0.12 0 0.60" rpy="0 0 0"/>
     </xacro:VLP-16>
   </xacro:if>
@@ -33,5 +33,5 @@
     </link>
     <joint name="surestar_joint" type="fixed">
-      <origin xyz="0.23 0.0 0.4" rpy="0.0 0.0 0.0"/>
+      <origin xyz="-0.12 0.0 0.6" rpy="0.0 0.0 0.0"/>
       <parent link="base_link"/>
       <child link="surestar"/>
@@ -73,5 +73,5 @@
     </gazebo>
   </xacro:if>
-  <xacro:include filename="$(find orne_box_description)/urdf/sensors/gnss.urdf.xacro"/> -->
+  <xacro:include filename="$(find orne_box_description)/urdf/sensors/gnss.urdf.xacro"/>
   <xacro:include filename="$(find orne_box_description)/urdf/sensors/camera.urdf.xacro"/>
   <xacro:sensor_gnss name="gnss" parent="base_link">

Commit message: first commit

File: orne_box_description/urdf/orne_box_3d_lidar_rfans.urdf.xacro (robot description, xacro)
@@ -8,5 +8,6 @@
     <!-- Setting for 3D-LiDAR -->
     <xacro:VLP-16 parent="base_link" name="surestar" topic="/rfans_points" organize_cloud="false" hz="10" samples="440" gpu="false">
-      <origin xyz="-0.12 0 0.60" rpy="0 0 0"/>
+      <origin xyz="-0.12 0 0.65" rpy="0 0 0"/>
+      <!--<origin xyz="-0.12 0 0.60" rpy="0 0 0"/>-->
     </xacro:VLP-16>
   </xacro:if>
